File: Hardware/RN41.brd (EAGLE design)
At the start: 25.4 x 22.9 mm, 8 parts, among them U1 BLUETOOTH-RN41"

Commit message: Production ready v15
Added fiducials and created panel
Parts:
- added FID1, FID2: FIDUCIALUFIDUCIAL, SparkFun-Aesthetics:MICRO-FIDUCIAL
