File: Hardware/RN41.sch (EAGLE design)
At the start: 8 parts, among them U1 BLUETOOTH-RN41"

Commit message: Production ready v15
Added fiducials and created panel
Parts:
- added FID1, FID2: FIDUCIALUFIDUCIAL, SparkFun-Aesthetics:FIDUCIALUFIDUCIAL
Changed lines of the file:
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@@
 <setting verticaltext="up"/>
 </settings>
-<grid distance="0.001" unitdist="inch" unit="inch" style="lines" multiple="1" display="yes" altdistance="0.01" altunitdist="inch" altunit="inch"/>
+<grid distance="0.1" unitdist="inch" unit="inch" style="lines" multiple="1" display="no" altdistance="0.01" altunitdist="inch" altunit="inch"/>
 <layers>
 <layer number="1" name="Top" color="4" fill="1" visible="no" active="no"/>
@@
 <part name="P+3" library="SparkFun" deviceset="VCC" device=""/>
 <part name="LOGO1" library="SparkFun-Aesthetics" deviceset="OSHW-LOGO" device="S"/>
+<part name="FID1" library="SparkFun-Aesthetics" deviceset="FIDUCIAL" device="UFIDUCIAL"/>
+<part name="FID2" library="SparkFun-Aesthetics" deviceset="FIDUCIAL" device="UFIDUCIAL"/>
 </parts>
 <sheets>
@@
 <instance part="P+3" gate="1" x="89.916" y="148.336"/>
 <instance part="LOGO1" gate="G$1" x="134.62" y="10.16"/>
+<instance part="FID1" gate="G$1" x="241.3" y="33.02"/>
+<instance part="FID2" gate="G$1" x="241.3" y="27.94"/>
 </instances>
 <busses>
